File: ExpansionBoards/KL25Z-Adapter/Pinscape Pico-KL25Z Adapter.brd (EAGLE design)
At the start: 81.9 x 53.5 mm, 17 parts, among them IC1 PCA9555APW,118, IC2 PCA9555APW,118, IC3 LIS3DHTR, IC30 ADS1115IDGSR, SW1 TS-1187A-B-A-B

Commit message: bug fixes
Connections:
- net 3V3_PICO: now also IC3.8
- net GND: no longer IC3.8
Routing:
- net 3V3_PICO: track 214.3 -> 216.7 mm
- net GND: track 29.7 -> 28.7 mm
Changed lines of the file:
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@@
 <signals>
 <signal name="GND">
-<contactref element="IC3" pad="8"/>
 <contactref element="IC3" pad="5"/>
 <contactref element="IC3" pad="10"/>
@@
 <contactref element="SW1" pad="D"/>
 <via x="39.05" y="24.55" extent="1-16" drill="0.3"/>
-<wire x1="60.25" y1="25.47" x2="60.25" y2="24.55" width="0.3" layer="1"/>
 <wire x1="60.25" y1="24.55" x2="60.5" y2="24.3" width="0.3" layer="1"/>
 <wire x1="58.55" y1="25.67" x2="57.57" y2="25.67" width="0.3" layer="1"/>
@@
 <wire x1="5.25" y1="40.7" x2="3.1" y2="42.85" width="1" layer="1"/>
 <wire x1="3.1" y1="44.675" x2="3.1" y2="42.85" width="1" layer="1"/>
+<contactref element="IC3" pad="8"/>
+<wire x1="60.25" y1="27.87" x2="60.25" y2="25.47" width="0.3" layer="1"/>
 </signal>
 <signal name="BUTTON1">
