File: ExpansionBoards/KL25Z-Adapter/PinscapePico KL25Z Adapter - PCA9555 vsn.brd (EAGLE design)
At the start: 81.9 x 53.5 mm, 17 parts, among them IC1 PCA9555APW,118, IC2 PCA9555APW,118, IC3 LIS3DHTR, IC30 ADS1115IDGSR, SW1 TS-1187A-B-A-B

Commit message: KL25Z adapter board updates;
Parts:
- added R6, R7: 4K, resistor:R1206
Connections:
- net 3V3_PICO: now also R6.1, R7.1
- net SCL: now also R7.2
- net SDA: now also R6.2
Routing:
- net 3V3_PICO: track 216.7 -> 227.1 mm
- net SCL: track 107.9 -> 114.0 mm
- net SDA: track 99.8 -> 105.8 mm
- net GND: track 28.7 -> 25.0 mm
Other:
- board size 81.9 x 53.5 mm -> 82.6 x 53.4 mm
- board text added: "REV 20250125"
- board text removed: "REV 20241118"

Commit message: KL25Z adapters - connect AGND to GND
Connections:
- net GND: now also RASPBERRY_PI_PICO.AGND
Changed lines of the file:
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@@
 <via x="66.15" y="25.15" extent="1-16" drill="0.3"/>
 <contactref element="IC1" pad="21"/>
+<contactref element="RASPBERRY_PI_PICO" pad="AGND"/>
 </signal>
 <signal name="SDA">
