File: ExpansionBoards/KL25Z-Adapter/PinscapePico KL25Z Adapter - PCA9555 vsn.sch (EAGLE design)
At the start: 17 parts, among them IC1 PCA9555APW,118, IC2 PCA9555APW,118, IC3 LIS3DHTR, IC30 ADS1115IDGSR, SW1 TS-1187A-B-A-B

Commit message: KL25Z adapter board updates;
Parts:
- added R6, R7: 4K, resistor:R-US_R1206
Connections:
- net 3V3_PICO: now also R6.1, R7.1
- net SCL: now also R7.2
- net SDA: now also R6.2
Other:
- note added: "Accelerometer I2C address 0x18 (001 1000)"
- note added: "I2C Address 0x20 (010 0000)"
- note added: "I2C Address 0x21 (010 0001)"
- note added: "I2C Bus Address 0x48 (100 1000)"
- note added: "I2C Pull-ups"
- note added: "KL25Z Header Connectors Install 0.1" pin sockets on BOTTOM of board"
- note removed: "Accelerometer I2C address 0x18"
- note removed: "I2C Address 0100000x ($20)"
- note removed: "I2C Address 0100001x ($21)"
- note removed: "I2C Bus Address $48 (1001000x)"
- moved on the sheet: C1, C2, LED1, R1, R2, R3, SW1

Commit message: KL25Z adapters - connect AGND to GND
Connections:
- net GND: now also RASPBERRY_PI_PICO.AGND
Changed lines of the file:
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@@
 <label x="48.26" y="119.38" size="1.27" layer="95" rot="R270" xref="yes"/>
+</segment>
+<segment>
+<pinref part="RASPBERRY_PI_PICO" gate="G$1" pin="AGND"/>
+<wire x1="71.12" y1="48.26" x2="73.66" y2="48.26" width="0.1524" layer="91"/>
+<label x="73.66" y="48.26" size="1.27" layer="95" xref="yes"/>
 </segment>
 </net>
