File: ExpansionBoards/DIY-Friendly/MainBoard/Pinscape Pico Expansion Board - DIY Friendly Main - Socketed Pico.brd (EAGLE design)
At the start: 160 x 107 mm, 115 parts, among them IC1 UCC27524P, IC10 ULN2803A, IC11 SN74HC165N, IC12 SN74HC165N, IC13 SN74HC74NE4, IC14 PC827, IC15 S-80833CLY, IC16 SN74HC165N, IC18 SN74HC165N, IC2 UCC27524P, IC3 UCC27524P, IC4 UCC27524P, IC5 UCC27524P, IC6 UCC27524P, IC7 ULN2803A, IC8 ULN2803A, IC9 ULN2803A, J1 30316-6002HB, J10 215079-4, J11 640454-2, J13 640445-2, J14 SSQ-108-02-T-S-RA, J2 640445-6, J3 640445-5, J4 640445-9, J5 1-640456-0, J6 1-640456-0, J7 1-640456-0, J8 1-640456-0, J9 30308-6002HB, Q1 FDPF085N10A, Q10 FDPF085N10A, Q11 FDPF085N10A, Q12 FDPF085N10A, Q13 BC337-25, Q15 2N5195G, Q16 2N2222A, Q2 FDPF085N10A, Q3 FDPF085N10A, Q4 FDPF085N10A, Q5 FDPF085N10A, Q6 FDPF085N10A, Q7 FDPF085N10A, Q8 FDPF085N10A, Q9 FDPF085N10A

Commit message: add tlc59116 wiring diagram to json doc; change Pro board IRED to constant-current circuit
Parts:
- R19: value 1.8K -> 540R
Changed lines of the file:
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@@
 <attribute name="VALUE" x="98.017" y="3.255" size="0.6" layer="27" align="center"/>
 </element>
-<element name="R19" library="resistor" package="0204/7" value="1.8K" x="97.3" y="14.7" smashed="yes">
+<element name="R19" library="resistor" package="0204/7" value="540R" x="97.3" y="14.7" smashed="yes">
 <attribute name="PARTNO" value="660-MFS1/4DCT52R47R0" x="97.3" y="14.7" size="0.6" layer="27" display="off"/>
 <attribute name="NAME" x="96.16" y="15.6954" size="0.9906" layer="25" ratio="10"/>
