File: ExpansionBoards/DIY-Friendly/MainBoard/Pinscape Pico Expansion Board - DIY Friendly Main - Socketed Pico.sch (EAGLE design)
At the start: 111 parts, among them IC1 UCC27524P, IC10 ULN2803A, IC11 SN74HC165N, IC12 SN74HC165N, IC13 SN74HC74NE4, IC14 PC827, IC15 S-80833CLY, IC16 SN74HC165N, IC18 SN74HC165N, IC2 UCC27524P, IC3 UCC27524P, IC4 UCC27524P, IC5 UCC27524P, IC6 UCC27524P, IC7 ULN2803A, IC8 ULN2803A, IC9 ULN2803A, J1 30316-6002HB, J10 215079-4, J11 640454-2, J13 640445-2, J14 SSQ-108-02-T-S-RA, J2 640445-6, J3 640445-5, J4 640445-9, J5 1-640456-0, J6 1-640456-0, J7 1-640456-0, J8 1-640456-0, J9 30308-6002HB, Q1 FDPF085N10A, Q10 FDPF085N10A, Q11 FDPF085N10A, Q12 FDPF085N10A, Q13 BC337-25, Q15 2N5195G, Q16 2N2222A, Q2 FDPF085N10A, Q3 FDPF085N10A, Q4 FDPF085N10A, Q5 FDPF085N10A, Q6 FDPF085N10A, Q7 FDPF085N10A, Q8 FDPF085N10A, Q9 FDPF085N10A

Commit message: add tlc59116 wiring diagram to json doc; change Pro board IRED to constant-current circuit
Parts:
- R19: value 1.8K -> 540R
Other:
- note added: "CURRENT-SENSE RESISTOR Resistor sets current to I(LED) = 0.5V/R R=2.5 ohms -> 200mA current"
- note added: "IR REMOTE CONTROL TRANSMITTER Use with TSAL6400 IRED or equivalent, with a peak wavelength around 940nm. Set the current-sense resistor according to the desired forward current on the IR LED. No external current-limiting resistor is needed. Two IR LEDs can be connected in series provided that Vf is less than about 1.9V."
- note removed: "IR REMOTE CONTROL TRANSMITTER Use with TSAL6400 IRED or equivalent, with a peak wavelength around 940nm. Set the current-sense resistor according to the desired forward current on the IR LED. The IR LED should be connected directly to the header (no external resistor is needed). Two IR LEDs can be connected in series provided that Vf is less than about 1.9V."
- note removed: "Resistor sets current to I(LED) = 0.5V/R R=2.5 ohms -> 200mA current"
Changed lines of the file:
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@@
 <part name="J11" library="SamacSys_Parts" deviceset="640454-2" device=""/>
 <part name="J10" library="SamacSys_Parts" deviceset="215079-4" device=""/>
-<part name="R19" library="resistor" deviceset="R-US_" device="0204/7" value="1.8K">
+<part name="R19" library="resistor" deviceset="R-US_" device="0204/7" value="540R">
 <attribute name="PARTNO" value="660-MFS1/4DCT52R47R0"/>
 </part>
@@
 <plain>
 <text x="12.7" y="76.2" size="1.778" layer="91">IR REMOTE CONTROL TRANSMITTER
-Use with TSAL6400 IRED or equivalent, with a
-peak wavelength around 940nm.  Set the
+Use with TSAL6400 IRED or equivalent, with
+a peak wavelength around 940nm.  Set the
 current-sense resistor according to the
 desired forward current on the IR LED.
-The IR LED should be connected directly to
-the header (no external resistor is needed).
+No external current-limiting resistor is
+needed.
 Two IR LEDs can be connected in series
 provided that Vf is less than about 1.9V.</text>
@@
 <text x="129.54" y="58.42" size="1.27" layer="91" align="top-left">Note: TE Connectivity Micro-Match 215079-4 base pairs
 with 215083-4 on-cable IDC connector.</text>
-<text x="53.34" y="17.78" size="1.778" layer="91" align="center-left">Resistor sets current to I(LED) = 0.5V/R
+<text x="53.34" y="17.78" size="1.778" layer="91" align="center-left">CURRENT-SENSE RESISTOR
+Resistor sets current to I(LED) = 0.5V/R
 R=2.5 ohms -&gt; 200mA current</text>
 <text x="60.96" y="33.02" size="1.778" layer="91" align="center-left">NPN substitutes: choose any medium-power NPN
 with Hfe around 100</text>
-<text x="63.5" y="106.68" size="1.778" layer="91">IR EMITTER / IR RECEIVER
+<text x="63.5" y="111.76" size="1.778" layer="91">IR EMITTER / IR RECEIVER
 The emitter and receiver are designed to be
 installed remotely to allow placing them in
