File: ExpansionBoards/DIY-Friendly/MainBoard/Pinscape Pico Expansion Board - DIY Friendly Main.sch (EAGLE design)
At the start: 111 parts, among them IC1 UCC27524P, IC10 ULN2803A, IC11 SN74HC165N, IC12 SN74HC165N, IC13 SN74HC74NE4, IC14 PC827, IC15 S-80833CLY, IC16 SN74HC165N, IC18 SN74HC165N, IC2 UCC27524P, IC3 UCC27524P, IC4 UCC27524P, IC5 UCC27524P, IC6 UCC27524P, IC7 ULN2803A, IC8 ULN2803A, IC9 ULN2803A, J1 30316-6002HB, J10 215079-4, J11 640454-2, J13 640445-2, J14 SSQ-108-02-T-S-RA, J2 640445-6, J3 640445-5, J4 640445-9, J5 1-640456-0, J6 1-640456-0, J7 1-640456-0, J8 1-640456-0, J9 30308-6002HB, Q1 STP19NF20, Q10 STP19NF20, Q11 STP19NF20, Q12 STP19NF20, Q13 BC337-25, Q15 2N5195G, Q16 2N2222A, Q2 FDPF085N10A, Q3 STP19NF20, Q4 STP19NF20, Q5 STP19NF20, Q6 STP19NF20, Q7 STP19NF20, Q8 STP19NF20, Q9 STP19NF20

Commit message: Exp boards: update gate resistors in BOMs
Other:
- note added: "Note: Gate resistor value of 200 Ohms is chosen to protect UCC27524P against damage due to excessive power dissipation during PWM switching. In principle, the gate resistor is primarily to suppress ringing, which only requires a small resistor in the 5 to 10 Ohm range. But practical testing suggests that UCC27524P may be vulnerable to overload when used with MOSFETs with high input capacitance (C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"
- note removed: "Note: Gate resistor value of 200 Ohms is chosen to protect UCC27524P against damage due to excessive power dissipation during PWM switching. In principle, the gate resistor is primarily to suppress ringing, which only requires a small resistor in the 5 to 10 Ohm range. But practical testing shows that UCC27524P is vulnerable to overload when used with MOSFETs with high input capacitance (C[ISS]).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"
Changed lines of the file:
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@@
 In principle, the gate resistor is primarily to suppress
 ringing, which only requires a small resistor in the 5
-to 10 Ohm range.  But practical testing shows that
-UCC27524P is vulnerable to overload when used
+to 10 Ohm range.  But practical testing suggests that
+UCC27524P may be vulnerable to overload when used
 with MOSFETs with high input capacitance (C[ISS]).
 200 Ohms appears safe for common FETs such as

Commit message: exp board: DIY: add errata to readme; reorient main board Flasher header silkscreen markings to match KL25Z expansion boards
Parts:
- J1: value 30316-6002HB -> 30316-6002HBROTATED; device SamacSys_Parts:30316-6002HB -> SamacSys_Parts:30316-6002HBROTATED
Changed lines of the file:
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@@
 <grid distance="0.1" unitdist="inch" unit="inch" style="lines" multiple="1" display="no" altdistance="0.01" altunitdist="inch" altunit="inch"/>
 <layers>
-<layer number="1" name="Top" color="4" fill="1" visible="no" active="no"/>
-<layer number="2" name="Route2" color="1" fill="3" visible="no" active="no"/>
-<layer number="3" name="Route3" color="4" fill="3" visible="no" active="no"/>
-<layer number="14" name="Route14" color="1" fill="6" visible="no" active="no"/>
-<layer number="15" name="Route15" color="4" fill="6" visible="no" active="no"/>
-<layer number="16" name="Bottom" color="1" fill="1" visible="no" active="no"/>
-<layer number="17" name="Pads" color="2" fill="1" visible="no" active="no"/>
-<layer number="18" name="Vias" color="2" fill="1" visible="no" active="no"/>
-<layer number="19" name="Unrouted" color="6" fill="1" visible="no" active="no"/>
-<layer number="20" name="Dimension" color="15" fill="1" visible="no" active="no"/>
-<layer number="21" name="tPlace" color="7" fill="1" visible="no" active="no"/>
-<layer number="22" name="bPlace" color="7" fill="1" visible="no" active="no"/>
-<layer number="23" name="tOrigins" color="15" fill="1" visible="no" active="no"/>
-<layer number="24" name="bOrigins" color="15" fill="1" visible="no" active="no"/>
-<layer number="25" name="tNames" color="7" fill="1" visible="no" active="no"/>
-<layer number="26" name="bNames" color="7" fill="1" visible="no" active="no"/>
-<layer number="27" name="tValues" color="7" fill="1" visible="no" active="no"/>
-<layer number="28" name="bValues" color="7" fill="1" visible="no" active="no"/>
+<layer number="1" name="Top" color="4" fill="1" visible="yes" active="no"/>
+<layer number="2" name="Route2" color="1" fill="3" visible="yes" active="no"/>
+<layer number="3" name="Route3" color="4" fill="3" visible="yes" active="no"/>
+<layer number="14" name="Route14" color="1" fill="6" visible="yes" active="no"/>
+<layer number="15" name="Route15" color="4" fill="6" visible="yes" active="no"/>
+<layer number="16" name="Bottom" color="1" fill="1" visible="yes" active="no"/>
+<layer number="17" name="Pads" color="2" fill="1" visible="yes" active="no"/>
+<layer number="18" name="Vias" color="2" fill="1" visible="yes" active="no"/>
+<layer number="19" name="Unrouted" color="6" fill="1" visible="yes" active="no"/>
+<layer number="20" name="Dimension" color="15" fill="1" visible="yes" active="no"/>
+<layer number="21" name="tPlace" color="7" fill="1" visible="yes" active="no"/>
+<layer number="22" name="bPlace" color="7" fill="1" visible="yes" active="no"/>
+<layer number="23" name="tOrigins" color="15" fill="1" visible="yes" active="no"/>
+<layer number="24" name="bOrigins" color="15" fill="1" visible="yes" active="no"/>
+<layer number="25" name="tNames" color="7" fill="1" visible="yes" active="no"/>
+<layer number="26" name="bNames" color="7" fill="1" visible="yes" active="no"/>
+<layer number="27" name="tValues" color="7" fill="1" visible="yes" active="no"/>
+<layer number="28" name="bValues" color="7" fill="1" visible="yes" active="no"/>
 <layer number="29" name="tStop" color="7" fill="3" visible="no" active="no"/>
 <layer number="30" name="bStop" color="7" fill="6" visible="no" active="no"/>
@@
 <layer number="35" name="tGlue" color="7" fill="4" visible="no" active="no"/>
 <layer number="36" name="bGlue" color="7" fill="5" visible="no" active="no"/>
-<layer number="37" name="tTest" color="7" fill="1" visible="no" active="no"/>
-<layer number="38" name="bTest" color="7" fill="1" visible="no" active="no"/>
+<layer number="37" name="tTest" color="7" fill="1" visible="yes" active="no"/>
+<layer number="38" name="bTest" color="7" fill="1" visible="yes" active="no"/>
 <layer number="39" name="tKeepout" color="4" fill="11" visible="no" active="no"/>
 <layer number="40" name="bKeepout" color="1" fill="11" visible="no" active="no"/>
@@
 <layer number="44" name="Drills" color="7" fill="1" visible="no" active="no"/>
 <layer number="45" name="Holes" color="7" fill="1" visible="no" active="no"/>
-<layer number="46" name="Milling" color="3" fill="1" visible="no" active="no"/>
-<layer number="47" name="Measures" color="7" fill="1" visible="no" active="no"/>
-<layer number="48" name="Document" color="7" fill="1" visible="no" active="no"/>
-<layer number="49" name="Reference" color="7" fill="1" visible="no" active="no"/>
-<layer number="50" name="dxf" color="7" fill="1" visible="no" active="no"/>
-<layer number="51" name="tDocu" color="7" fill="1" visible="no" active="no"/>
-<layer number="52" name="bDocu" color="7" fill="1" visible="no" active="no"/>
-<layer number="53" name="tPadExt" color="7" fill="1" visible="no" active="no"/>
-<layer number="54" name="bPadExt" color="1" fill="1" visible="no" active="no"/>
-<layer number="56" name="wert" color="7" fill="1" visible="no" active="no"/>
-<layer number="57" name="tCAD" color="7" fill="1" visible="no" active="no"/>
-<layer number="58" name="b3D" color="7" fill="1" visible="no" active="no"/>
-<layer number="59" name="tCarbon" color="7" fill="1" visible="no" active="no"/>
-<layer number="60" name="bCarbon" color="7" fill="1" visible="no" active="no"/>
-<layer number="61" name="stand" color="7" fill="1" visible="no" active="no"/>
+<layer number="46" name="Milling" color="3" fill="1" visible="yes" active="no"/>
+<layer number="47" name="Measures" color="7" fill="1" visible="yes" active="no"/>
+<layer number="48" name="Document" color="7" fill="1" visible="yes" active="no"/>
+<layer number="49" name="Reference" color="7" fill="1" visible="yes" active="no"/>
+<layer number="50" name="dxf" color="7" fill="1" visible="yes" active="no"/>
+<layer number="51" name="tDocu" color="7" fill="1" visible="yes" active="no"/>
+<layer number="52" name="bDocu" color="7" fill="1" visible="yes" active="no"/>
+<layer number="53" name="tPadExt" color="7" fill="1" visible="yes" active="no"/>
+<layer number="54" name="bPadExt" color="1" fill="1" visible="yes" active="no"/>
+<layer number="56" name="wert" color="7" fill="1" visible="yes" active="no"/>
+<layer number="57" name="tCAD" color="7" fill="1" visible="yes" active="no"/>
+<layer number="58" name="b3D" color="7" fill="1" visible="yes" active="no"/>
+<layer number="59" name="tCarbon" color="7" fill="1" visible="yes" active="no"/>
+<layer number="60" name="bCarbon" color="7" fill="1" visible="yes" active="no"/>
+<layer number="61" name="stand" color="7" fill="1" visible="yes" active="no"/>
 <layer number="88" name="SimResults" color="9" fill="1" visible="yes" active="yes"/>
 <layer number="89" name="SimProbes" color="9" fill="1" visible="yes" active="yes"/>
@@
 <part name="IC9" library="uln-udn" deviceset="ULN2803A" device="" value="ULN2803A"/>
 <part name="IC10" library="uln-udn" deviceset="ULN2803A" device="" value="ULN2803A"/>
-<part name="J1" library="SamacSys_Parts" deviceset="30316-6002HB" device=""/>
+<part name="J1" library="SamacSys_Parts" deviceset="30316-6002HB" device="ROTATED" value="30316-6002HBROTATED"/>
 <part name="J12" library="pinhead" deviceset="PINHD-1X3" device=""/>
 <part name="IC5" library="SamacSys_Parts" deviceset="UCC27524P" device=""/>

Commit message: exp board: DIY power: add guard ring and isolated ground plane under DS1307 crystal per App Note 58
Other:
- note added: "AIN0"
- note added: "AIN3"
- moved on the sheet: JP3, JP4

Commit message: Exp board: DIY main: improve reference designator ordering, fix bypass cap proximities to shift register chips, silkscreen cleanup
Parts:
- removed C19: 100nF, rcl:C-US025-024X044
- added C17: 100nF, rcl:C-US025-024X044
- C10, C7: value 100nF -> 4.7uF; PARTNO K104K15X7RF5TL2 -> 810-FG14X5R1H475KRT0
- C16, C8: value 4.7uF -> 100nF; PARTNO 810-FG14X5R1H475KRT0 -> K104K15X7RF5TL2
- IC11: value SN74HC165N -> SN74HC74NE4; device SamacSys_Parts:SN74HC165N -> SamacSys_Parts:SN74HC74NE4
- IC12: value SN74HC165N -> S-80833CLY; device SamacSys_Parts:SN74HC165N -> SamacSys_Parts:S-80833CLY-B2-UTO92
- IC13: value SN74HC74NE4 -> PC827; device SamacSys_Parts:SN74HC74NE4 -> optocoupler:PC827
- IC14: value PC827 -> SN74HC165N; device optocoupler:PC827 -> SamacSys_Parts:SN74HC165N
- IC15: value S-80833CLY -> SN74HC165N; device SamacSys_Parts:S-80833CLY-B2-UTO92 -> SamacSys_Parts:SN74HC165N
- renumbered IC18 to IC17
Connections:
- net 12V: now also C10.2, C9.2; no longer C13.2, C14.2
- net 3V3_PICO: now also C15.2, C16.2, C17.2, IC13B.COL, IC14.VCC, IC15.VCC; no longer C10.2, C19.2, C9.2, IC11.VCC, IC12.VCC, IC14B.COL
- net 5V: now also C13.1, C14.1, IC11.1!PRE, IC11.1D, IC11.VCC, IC12.VDD, IC13A.COL; no longer C15.1, C16.1, IC13.1!PRE, IC13.1D, IC13.VCC, IC14A.COL, IC15.VDD
- net BUTTON1: now also IC14.A; no longer IC11.A
- net BUTTON10: now also IC15.B; no longer IC12.B
- net BUTTON11: now also IC15.C; no longer IC12.C
- net BUTTON12: now also IC15.D; no longer IC12.D
- net BUTTON13: now also IC15.H; no longer IC12.H
- net BUTTON14: now also IC15.G; no longer IC12.G
- net BUTTON15: now also IC15.F; no longer IC12.F
- net BUTTON16: now also IC15.E; no longer IC12.E
- net BUTTON2: now also IC14.B; no longer IC11.B
- net BUTTON3: now also IC14.C; no longer IC11.C
- net BUTTON4: now also IC14.D; no longer IC11.D
- net BUTTON5: now also IC14.H; no longer IC11.H
- net BUTTON6: now also IC14.G; no longer IC11.G
- net BUTTON7: now also IC14.F; no longer IC11.F
- net BUTTON8: now also IC14.E; no longer IC11.E
- net BUTTON9: now also IC15.A; no longer IC12.A
- net BUTTON_CLK: now also IC14.CLK, IC15.CLK; no longer IC11.CLK, IC12.CLK
- net BUTTON_DATA: now also IC14.QH; no longer IC11.QH
- net BUTTON_SHLD: now also IC14.SH/!LD, IC15.SH/!LD; no longer IC11.SH/!LD, IC12.SH/!LD
- net GND: now also C13.2, C14.2, C15.1, C16.1, C17.1, IC14.CLK_INH, IC14.GND, IC15.CLK_INH; no longer C13.1, C14.1, C15.2, C16.2, C19.1, IC11.CLK_INH, IC12.CLK_INH, IC13.GND
- net N$21: now also IC14.SER, IC15.QH; no longer IC11.SER, IC12.QH
- net N$22: now also IC15.SER; no longer IC12.SER
- net N$58: now also IC11.1CLK, IC13A.EMIT; no longer IC13.1CLK, IC14A.EMIT
- net N$59: now also IC13A.C; no longer IC14A.C
- net N$63: now also IC11.!1CLR, IC12.OUT; no longer IC13.!1CLR, IC15.OUT
- net N$65: now also IC13B.C; no longer IC14B.C
- net N$68: now also IC11.1Q, IC13B.A; no longer IC13.1Q, IC14B.A
- net PSU2_STATUS_SENSE: now also IC13B.EMIT; no longer IC14B.EMIT
- net PSU2_STATUS_SET: now also IC13A.A; no longer IC14A.A

Commit message: exp board: update BOM for MOSFET recommendations
Parts:
- added JP5: (no value), pinhead:PINHD-1X8
Connections:
- net 3V3_PERIPHERAL: now also JP5.1
- net ACCEL_INTR: now also JP5.5
- net GND: now also JP5.2
- net SCL: now also JP5.6
- net SDA: now also JP5.7
Other:
- note added: "Adafruit MMA8451Q Module"
- note added: "INTR2 (NC)"
- note added: "Install one 8x1 pin 0.1" socket on this board Install one 8x1 pin 0.1" pin header on BOTTOM of Adafruit MMA8451Q module Plug MMA8451Q module into sockets"
Changed lines of the file:
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@@
 <part name="GND7" library="supply1" deviceset="GND" device=""/>
 <part name="J14" library="SamacSys_Parts" deviceset="SSQ-108-02-T-S-RA" device=""/>
+<part name="JP5" library="pinhead" deviceset="PINHD-1X8" device=""/>
 </parts>
 <sheets>
@@
 <text x="129.54" y="50.8" size="1.778" layer="97" align="center-left">&lt;== Must be ADC-capable</text>
 <text x="48.006" y="27.94" size="1.778" layer="97" rot="R180" align="center-left">Must be an I2C0 SDA pin ==&gt;</text>
-<text x="165.1" y="40.64" size="2.54" layer="91" align="center-left">Main Pico Hard Reset</text>
+<text x="172.72" y="35.56" size="2.54" layer="91" align="center-left">Main Pico Hard Reset</text>
 <text x="91.44" y="109.22" size="2.54" layer="91" align="center">Status LED</text>
 <text x="195.58" y="109.22" size="2.54" layer="91" align="center">3.3V Peripheral Power</text>
@@
 <description>Accelerometer</description>
 <plain>
-<text x="60.96" y="46.228" size="2.54" layer="91" align="center">Adafruit LIS3DH Module</text>
+<text x="60.96" y="43.688" size="2.54" layer="91" align="center">Adafruit LIS3DH Module</text>
 <text x="60.96" y="35.56" size="1.905" layer="91" align="center">Install two 6x1 pin 0.1" sockets on this board
 Install two 6x1 pin 0.1" pin headers on BOTTOM of Adafruit LIS3DH module
@@
 I2C address $18</text>
 <text x="40.64" y="5.08" size="1.27" layer="95" align="center-right">CS High=I2C mode</text>
+<text x="63.5" y="102.108" size="2.54" layer="91" align="center">Adafruit MMA8451Q Module</text>
+<text x="63.5" y="93.98" size="1.905" layer="91" align="center">Install one 8x1 pin 0.1" socket on this board
+Install one 8x1 pin 0.1" pin header on BOTTOM of Adafruit MMA8451Q module
+Plug MMA8451Q module into sockets</text>
+<text x="78.74" y="76.2" size="1.27" layer="95" align="center-right">3V3 OUT (NC)</text>
+<text x="78.74" y="73.66" size="1.27" layer="95" align="center-right">INTR2 (NC)</text>
 </plain>
 <instances>
 <instance part="JP1" gate="A" x="50.8" y="12.7"/>
 <instance part="JP2" gate="A" x="86.36" y="12.7"/>
+<instance part="JP5" gate="A" x="86.36" y="71.12"/>
 </instances>
 <busses>
@@
 <label x="76.2" y="15.24" size="1.27" layer="95" rot="R180" xref="yes"/>
 </segment>
+<segment>
+<pinref part="JP5" gate="A" pin="2"/>
+<wire x1="76.2" y1="78.74" x2="83.82" y2="78.74" width="0.1524" layer="91"/>
+<label x="76.2" y="78.74" size="1.27" layer="95" rot="R180" xref="yes"/>
+</segment>
 </net>
 <net name="SCL" class="0">
@@
 <label x="76.2" y="12.7" size="1.27" layer="95" rot="R180" xref="yes"/>
 </segment>
+<segment>
+<pinref part="JP5" gate="A" pin="6"/>
+<wire x1="76.2" y1="68.58" x2="83.82" y2="68.58" width="0.1524" layer="91"/>
+<label x="76.2" y="68.58" size="1.27" layer="95" rot="R180" xref="yes"/>
+</segment>
 </net>
 <net name="SDA" class="0">
@@
 <label x="76.2" y="10.16" size="1.27" layer="95" rot="R180" xref="yes"/>
 </segment>
+<segment>
+<pinref part="JP5" gate="A" pin="7"/>
+<wire x1="76.2" y1="66.04" x2="83.82" y2="66.04" width="0.1524" layer="91"/>
+<label x="76.2" y="66.04" size="1.27" layer="95" rot="R180" xref="yes"/>
+</segment>
 </net>
 <net name="ACCEL_INTR" class="0">
@@
 <label x="76.2" y="7.62" size="1.27" layer="95" rot="R180" xref="yes"/>
 </segment>
+<segment>
+<pinref part="JP5" gate="A" pin="5"/>
+<wire x1="76.2" y1="71.12" x2="83.82" y2="71.12" width="0.1524" layer="91"/>
+<label x="76.2" y="71.12" size="1.27" layer="95" rot="R180" xref="yes"/>
+</segment>
 </net>
 <net name="3V3_PERIPHERAL" class="0">
@@
 <label x="40.64" y="7.62" size="1.27" layer="95" rot="R180" xref="yes"/>
 </segment>
-</net>
+<segment>
+<pinref part="JP5" gate="A" pin="1"/>
+<wire x1="76.2" y1="81.28" x2="83.82" y2="81.28" width="0.1524" layer="91"/>
+<label x="76.2" y="81.28" size="1.27" layer="95" rot="R180" xref="yes"/>
+</segment>
+</net>

Commit message: Improve expansion board IR receiver documentation
Other:
- note added: "IR REMOTE CONTROL TRANSMITTER Use with VSLB4940, TSAL6400, or a similar IR LED with a peak wavelength around 940nm. Set the current-sense resistor according to the desired forward current on the IR LED. Set to 200 mA for VSLB4940 or TSAL6400; for others, use a current between the "continuous" and "peak" I(F) values listed in the Absolute Maximum Values section of the data sheet. No external curre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"
- note removed: "IR REMOTE CONTROL TRANSMITTER Use with TSAL6400 IRED or equivalent, with a peak wavelength around 940nm. Set the current-sense resistor according to the desired forward current on the IR LED. No external current-limiting resistor is needed. Two IR LEDs can be connected in series provided that Vf is less than about 1.9V."
Changed lines of the file:
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@@
 <plain>
 <text x="12.7" y="76.2" size="1.778" layer="91">IR REMOTE CONTROL TRANSMITTER
-Use with TSAL6400 IRED or equivalent, with
-a peak wavelength around 940nm.  Set the
-current-sense resistor according to the
-desired forward current on the IR LED.
+Use with VSLB4940, TSAL6400, or a similar
+IR LED with a peak wavelength around
+940nm.  Set the current-sense resistor
+according to the desired forward current
+on the IR LED.  Set to 200 mA for VSLB4940
+or TSAL6400; for others, use a current
+between the "continuous" and "peak" I(F)
+values listed in the Absolute Maximum
+Values section of the data sheet.
 No external current-limiting resistor is
 needed.
@@
 <text x="60.96" y="33.02" size="1.778" layer="91" align="center-left">NPN substitutes: choose any medium-power NPN
 with Hfe around 100</text>
-<text x="63.5" y="111.76" size="1.778" layer="91">IR EMITTER / IR RECEIVER
+<text x="63.5" y="124.46" size="1.778" layer="91">IR EMITTER / IR RECEIVER
 The emitter and receiver are designed to be
 installed remotely to allow placing them in

Commit message: exp boards: DIY-friendly main: add button header pin labels; add button header pin label diagram to readme
Parts:
- C7: value 4.7uF -> 100nF; PARTNO 810-FG14X5R1H475KRT0 -> K104K15X7RF5TL2
- C8: value 100nF -> 4.7uF; PARTNO K104K15X7RF5TL2 -> 810-FG14X5R1H475KRT0
Other:
- moved on the sheet: C7, C8, J12, J14, J2, QWIIC1G$1
