File: ExpansionBoards/DIY-Friendly/PowerBoard/Pinscape Pico Expansion Board - DIY Friendly Power.sch (EAGLE design)
At the start: 83 parts, among them IC1 UCC27524P, IC10 ULN2803A, IC11 ULN2803A, IC12 ULN2803A, IC13 DS1307+, IC2 UCC27524P, IC3 UCC27524P, IC4 UCC27524P, IC5 UCC27524P, IC6 UCC27524P, IC7 UCC27524P, IC8 UCC27524P, IC9 ULN2803A, J1 640445-9, J2 640445-9, J3 640445-6, J4 1-640456-0, J5 1-640456-0, J6 1-640456-0, J7 1-640456-0, Q1 FDPF085N10A, Q10 FDPF085N10A, Q11 FDPF085N10A, Q12 FDPF085N10A, Q13 FDPF085N10A, Q14 FDPF085N10A, Q15 FDPF085N10A, Q16 FDPF085N10A, Q17 2N2222A, Q18 2N2222A, Q2 FDPF085N10A, Q3 FDPF085N10A, Q4 FDPF085N10A, Q5 FDPF085N10A, Q6 FDPF085N10A, Q7 FDPF085N10A, Q8 FDPF085N10A, Q9 FDPF085N10A, Y1 ECS-.327-12.5-13X-C

Commit message: PCB parts lists (BOMs); power distro board edits
Other:
- note added: "Copyright and License Info Pinscape Pico DIY Friendly Expansion Board (Power Board) Copyright 2024, 2025 Michael J Roberts BSD 3-clause license"
Changed lines of the file:
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@@
+</nets>
+</sheet>
+<sheet>
+<description>Notes</description>
+<plain>
+<text x="5.08" y="5.08" size="2.54" layer="91">Copyright and License Info
+  Pinscape Pico DIY Friendly Expansion Board (Power Board)
+  Copyright 2024, 2025 Michael J Roberts
+  BSD 3-clause license</text>
+</plain>
+<instances>
+</instances>
+<busses>
+</busses>
+<nets>
 </nets>
 </sheet>

Commit message: BOM tweaks
Parts:
- Q1, Q10, Q11, Q12, Q13, Q14, Q15, Q16, Q2, Q3, Q4, Q5, Q6, Q7, Q8, Q9: value FDPF085N10A -> STP19NF20
- R1, R10, R11, R12, R14, R15, R16, R17, R2, R3, R4, R5, R6, R7, R8, R9: value 4R7 -> 200R
Other:
- note added: "Note: Gate resistor value of 200 Ohms is chosen to protect UCC27524P against damage due to excessive power dissipation during PWM switching. In principle, the gate resistor is primarily to suppress ringing, which only requires a small resistor in the 5 to 10 Ohm range. But practical testing shows that UCC27524P is vulnerable to overload when used with MOSFETs with high input capacitance (C[ISS]).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"
- note added: "Note: Many similar MOSFETs are available. Choose a TO-220 package with G-D-S pin order and Absolute Maximum V[gs] of at least +/- 20V. Low input capacitance (C[ISS]) and total gate charge (Q[g]) are also desirable. Beyond that, choose based on the required Absolute Maximum values for drain current and voltage (I[D], V[DS]), which determine the limits for the output devices you can connect to the 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"
