File: ExpansionBoards/PowerDistribution/Power Distribution Board.sch (EAGLE design)
At the start: 47 parts, among them J1 216571-2005, J10 640445-6, J11 640445-6, J12 640445-5, J13 640445-2, J14 640445-4, J15 640445-3, J16 216571-2003, J17 640445-8, J2 216571-2002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

Commit message: exp board: power distro tweaks
Parts:
- removed J1, J3: 216571-2005, SamacSys_Parts:216571-2005
- added J18, J19: 206832-0601, SamacSys_Parts:206832-0601
Connections:
- net 24V: now also J18.5, J18.6; no longer J3.2
- net GND: now also J18.1, J18.4, J19.1, J19.4; no longer J1.1, J1.3, J3.1, J3.3
- net LINE_HOT: now also J18.3, J19.3; no longer J1.5, J3.5
- net LINE_NEUTRAL: now also J18.2, J19.2; no longer J1.4, J3.4
- net N$1: now also J19.5, J19.6; no longer J1.2
Changed lines of the file:
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@@
 <attribute name="TYPE" value="Tantalum"/>
 </part>
-<part name="J3" library="SamacSys_Parts" deviceset="216571-2005" device=""/>
-<part name="J1" library="SamacSys_Parts" deviceset="216571-2005" device=""/>
 <part name="J2" library="SamacSys_Parts" deviceset="216571-2002" device=""/>
 <part name="K1" library="SamacSys_Parts" deviceset="AHQSS105DM2FA0G" device=""/>
@@
 <part name="J12" library="SamacSys_Parts" deviceset="640445-5" device=""/>
 <part name="J14" library="SamacSys_Parts" deviceset="640445-4" device=""/>
+<part name="J18" library="SamacSys_Parts" deviceset="206832-0601" device=""/>
+<part name="J19" library="SamacSys_Parts" deviceset="206832-0601" device=""/>
 </parts>
 <sheets>
@@
 </plain>
 <instances>
-<instance part="J3" gate="G$1" x="33.02" y="38.1" smashed="yes">
-<attribute name="NAME" x="49.53" y="38.1" size="1.778" layer="95" align="center-left"/>
-<attribute name="VALUE" x="49.53" y="35.56" size="1.778" layer="96" align="center-left"/>
-</instance>
 <instance part="LED4" gate="G$1" x="38.1" y="7.62" rot="R90"/>
 <instance part="R10" gate="G$1" x="27.94" y="7.62" smashed="yes" rot="R180">
@@
 <attribute name="VALUE" x="34.798" y="5.588" size="1.778" layer="96" rot="R180"/>
 </instance>
+<instance part="J18" gate="G$1" x="33.02" y="38.1"/>
 </instances>
 <busses>
@@
 <net name="LINE_HOT" class="0">
 <segment>
-<pinref part="J3" gate="G$1" pin="5"/>
 <wire x1="27.94" y1="38.1" x2="33.02" y2="38.1" width="0.1524" layer="91"/>
 <label x="27.94" y="38.1" size="1.27" layer="95" rot="R180" xref="yes"/>
+<pinref part="J18" gate="G$1" pin="3"/>
 </segment>
 </net>
 <net name="LINE_NEUTRAL" class="0">
 <segment>
-<pinref part="J3" gate="G$1" pin="4"/>
 <wire x1="27.94" y1="35.56" x2="33.02" y2="35.56" width="0.1524" layer="91"/>
 <label x="27.94" y="35.56" size="1.27" layer="95" rot="R180" xref="yes"/>
+<pinref part="J18" gate="G$1" pin="2"/>
 </segment>
 </net>
 <net name="GND" class="0">
 <segment>
-<label x="27.94" y="27.94" size="1.27" layer="95" rot="R180" xref="yes"/>
-<pinref part="J3" gate="G$1" pin="1"/>
-<wire x1="33.02" y1="27.94" x2="27.94" y2="27.94" width="0.1524" layer="91"/>
+<label x="58.42" y="33.02" size="1.27" layer="95" xref="yes"/>
+<pinref part="J18" gate="G$1" pin="4"/>
+<wire x1="53.34" y1="33.02" x2="58.42" y2="33.02" width="0.1524" layer="91"/>
 </segment>
 <segment>
 <label x="27.94" y="33.02" size="1.27" layer="95" rot="R180" xref="yes"/>
-<pinref part="J3" gate="G$1" pin="3"/>
 <wire x1="27.94" y1="33.02" x2="33.02" y2="33.02" width="0.1524" layer="91"/>
+<pinref part="J18" gate="G$1" pin="1"/>
 </segment>
 <segment>
@@
 <net name="24V" class="0">
 <segment>
-<label x="27.94" y="30.48" size="1.27" layer="95" rot="R180" xref="yes"/>
-<pinref part="J3" gate="G$1" pin="2"/>
-<wire x1="27.94" y1="30.48" x2="33.02" y2="30.48" width="0.1524" layer="91"/>
+<label x="58.42" y="38.1" size="1.27" layer="95" xref="yes"/>
+<wire x1="58.42" y1="38.1" x2="55.88" y2="38.1" width="0.1524" layer="91"/>
+<pinref part="J18" gate="G$1" pin="6"/>
+<pinref part="J18" gate="G$1" pin="5"/>
+<wire x1="55.88" y1="38.1" x2="53.34" y2="38.1" width="0.1524" layer="91"/>
+<wire x1="53.34" y1="35.56" x2="55.88" y2="35.56" width="0.1524" layer="91"/>
+<wire x1="55.88" y1="35.56" x2="55.88" y2="38.1" width="0.1524" layer="91"/>
+<junction x="55.88" y="38.1"/>
 </segment>
 <segment>
@@
 <description>48V SMPS</description>
 <plain>
-<text x="111.76" y="111.76" size="1.778" layer="91" align="center">48V SMPS</text>
+<text x="53.34" y="96.52" size="1.778" layer="91" align="center">48V SMPS</text>
 <text x="119.38" y="60.96" size="1.778" layer="91">COIN DOOR INTERLOCK
 5V control signal to coin door switch
@@
 Serves as indicator, and
 drains caps when power is off.</text>
-<text x="83.058" y="98.806" size="1.778" layer="91" align="center-right">+48V DC</text>
+<text x="81.28" y="92.964" size="1.778" layer="91" align="center-right">+48V DC</text>
 </plain>
 <instances>
-<instance part="J1" gate="G$1" x="101.6" y="106.68" smashed="yes">
-<attribute name="NAME" x="118.11" y="106.68" size="1.778" layer="95" align="center-left"/>
-<attribute name="VALUE" x="118.11" y="104.14" size="1.778" layer="96" align="center-left"/>
-</instance>
 <instance part="J2" gate="G$1" x="132.08" y="53.34" smashed="yes">
 <attribute name="NAME" x="148.59" y="53.34" size="1.778" layer="95" align="center-left"/>
@@
 <attribute name="VALUE" x="106.68" y="47.244" size="1.778" layer="96"/>
 </instance>
+<instance part="J19" gate="G$1" x="45.72" y="91.44" smashed="yes">
+<attribute name="NAME" x="49.53" y="81.28" size="1.778" layer="95" align="center-left"/>
+<attribute name="VALUE" x="49.53" y="78.74" size="1.778" layer="96" align="center-left"/>
+</instance>
 </instances>
 <busses>
@@
 <net name="LINE_HOT" class="0">
 <segment>
-<label x="99.06" y="106.68" size="1.27" layer="95" rot="R180" xref="yes"/>
-<pinref part="J1" gate="G$1" pin="5"/>
-<wire x1="101.6" y1="106.68" x2="99.06" y2="106.68" width="0.1524" layer="91"/>
+<label x="43.18" y="91.44" size="1.27" layer="95" rot="R180" xref="yes"/>
+<pinref part="J19" gate="G$1" pin="3"/>
+<wire x1="43.18" y1="91.44" x2="45.72" y2="91.44" width="0.1524" layer="91"/>
 </segment>
 </net>
 <net name="LINE_NEUTRAL" class="0">
 <segment>
-<label x="99.06" y="104.14" size="1.27" layer="95" rot="R180" xref="yes"/>
-<pinref part="J1" gate="G$1" pin="4"/>
-<wire x1="101.6" y1="104.14" x2="99.06" y2="104.14" width="0.1524" layer="91"/>
+<label x="43.18" y="88.9" size="1.27" layer="95" rot="R180" xref="yes"/>
+<pinref part="J19" gate="G$1" pin="2"/>
+<wire x1="43.18" y1="88.9" x2="45.72" y2="88.9" width="0.1524" layer="91"/>
 </segment>
 </net>
 <net name="GND" class="0">
-<segment>
-<pinref part="J1" gate="G$1" pin="1"/>
-<wire x1="99.06" y1="96.52" x2="101.6" y2="96.52" width="0.1524" layer="91"/>
-<label x="99.06" y="96.52" size="1.27" layer="95" rot="R180" xref="yes"/>
-</segment>
 <segment>
 <pinref part="C5" gate="G$1" pin="-"/>
@@
 </segment>
 <segment>
-<label x="99.06" y="101.6" size="1.27" layer="95" rot="R180" xref="yes"/>
-<pinref part="J1" gate="G$1" pin="3"/>
-<wire x1="99.06" y1="101.6" x2="101.6" y2="101.6" width="0.1524" layer="91"/>
+<label x="43.18" y="86.36" size="1.27" layer="95" rot="R180" xref="yes"/>
+<pinref part="J19" gate="G$1" pin="1"/>
+<wire x1="43.18" y1="86.36" x2="45.72" y2="86.36" width="0.1524" layer="91"/>
 </segment>
 <segment>
@@
 <wire x1="93.98" y1="45.72" x2="93.98" y2="43.18" width="0.1524" layer="91"/>
 <label x="93.98" y="43.18" size="1.27" layer="95" xref="yes"/>
+</segment>
+<segment>
+<pinref part="J19" gate="G$1" pin="4"/>
+<wire x1="66.04" y1="86.36" x2="68.58" y2="86.36" width="0.1524" layer="91"/>
+<label x="68.58" y="86.36" size="1.27" layer="95" xref="yes"/>
 </segment>
 </net>
@@
 <net name="N$1" class="0">
 <segment>
-<pinref part="J1" gate="G$1" pin="2"/>
-<wire x1="101.6" y1="99.06" x2="83.82" y2="99.06" width="0.1524" layer="91"/>
-<wire x1="83.82" y1="99.06" x2="83.82" y2="91.44" width="0.1524" layer="91"/>
 <pinref part="Q2" gate="G$1" pin="S"/>
 <pinref part="R7" gate="G$1" pin="1"/>
-<wire x1="83.82" y1="91.44" x2="83.82" y2="83.82" width="0.1524" layer="91"/>
+<wire x1="83.82" y1="91.44" x2="83.82" y2="88.9" width="0.1524" layer="91"/>
+<wire x1="83.82" y1="88.9" x2="83.82" y2="83.82" width="0.1524" layer="91"/>
 <wire x1="93.98" y1="88.9" x2="93.98" y2="91.44" width="0.1524" layer="91"/>
 <wire x1="93.98" y1="91.44" x2="83.82" y2="91.44" width="0.1524" layer="91"/>
 <junction x="83.82" y="91.44"/>
-</segment>
-</net>
+<pinref part="J19" gate="G$1" pin="6"/>
+<wire x1="66.04" y1="91.44" x2="83.82" y2="91.44" width="0.1524" layer="91"/>
+<pinref part="J19" gate="G$1" pin="5"/>
+<wire x1="66.04" y1="88.9" x2="83.82" y2="88.9" width="0.1524" layer="91"/>
+<junction x="83.82" y="88.9"/>
+</segment>
+</net>
